Commit message: fix: srdf

File: ur_moveit_config/srdf/ur_macro.srdf.xacro (robot description, xacro)
@@ -12,45 +12,45 @@
     <!--SUBGROUPS - Groups can also be formed by referencing to already defined group names-->
     <group name="ur_manipulator">
-      <chain base_link="base_link" tip_link="tool0" />
+      <chain base_link="ur_base_link" tip_link="ur_tool0" />
     </group>
     <!--GROUP STATES - Purpose - Define a named state for a particular group, in terms of joint values. This is useful to define states like 'folded arms'-->
     <group_state name="home" group="ur_manipulator">
-      <joint name="elbow_joint" value="0" />
-      <joint name="shoulder_lift_joint" value="-1.5707" />
-      <joint name="shoulder_pan_joint" value="0" />
-      <joint name="wrist_1_joint" value="0" />
-      <joint name="wrist_2_joint" value="0" />
-      <joint name="wrist_3_joint" value="0" />
+      <joint name="ur_elbow_joint" value="0" />
+      <joint name="ur_shoulder_lift_joint" value="-1.5707" />
+      <joint name="ur_shoulder_pan_joint" value="0" />
+      <joint name="ur_wrist_1_joint" value="0" />
+      <joint name="ur_wrist_2_joint" value="0" />
+      <joint name="ur_wrist_3_joint" value="0" />
     </group_state>
     <group_state name="up" group="ur_manipulator">
-      <joint name="elbow_joint" value="0" />
-      <joint name="shoulder_lift_joint" value="-1.5707" />
-      <joint name="shoulder_pan_joint" value="0" />
-      <joint name="wrist_1_joint" value="-1.5707" />
-      <joint name="wrist_2_joint" value="0" />
-      <joint name="wrist_3_joint" value="0" />
+      <joint name="ur_elbow_joint" value="0" />
+      <joint name="ur_shoulder_lift_joint" value="-1.5707" />
+      <joint name="ur_shoulder_pan_joint" value="0" />
+      <joint name="ur_wrist_1_joint" value="-1.5707" />
+      <joint name="ur_wrist_2_joint" value="0" />
+      <joint name="ur_wrist_3_joint" value="0" />
     </group_state>
     <group_state name="test_configuration" group="ur_manipulator">
-      <joint name="elbow_joint" value="1.4" />
-      <joint name="shoulder_lift_joint" value="-1.62" />
-      <joint name="shoulder_pan_joint" value="1.54" />
-      <joint name="wrist_1_joint" value="-1.2" />
-      <joint name="wrist_2_joint" value="-1.6" />
-      <joint name="wrist_3_joint" value="-0.11" />
+      <joint name="ur_elbow_joint" value="1.4" />
+      <joint name="ur_shoulder_lift_joint" value="-1.62" />
+      <joint name="ur_shoulder_pan_joint" value="1.54" />
+      <joint name="ur_wrist_1_joint" value="-1.2" />
+      <joint name="ur_wrist_2_joint" value="-1.6" />
+      <joint name="ur_wrist_3_joint" value="-0.11" />
     </group_state>
     <!--END EFFECTOR - Purpose - Represent information about an end effector.-->
     <!--VIRTUAL JOINT - Purpose - this element defines a virtual joint between a robot link and an external frame of reference (considered fixed with respect to the robot)-->
     <!--DISABLE COLLISIONS - By default it is assumed that any link of the robot could potentially come into collision with any other link in the robot. This tag disables collision checking between a specified pair of links. -->
-    <disable_collisions link1="base_link" link2="base_link_inertia" reason="Adjacent" />
-    <disable_collisions link1="base_link_inertia" link2="shoulder_link" reason="Adjacent" />
-    <disable_collisions link1="tool0" link2="wrist_1_link" reason="Never" />
-    <disable_collisions link1="tool0" link2="wrist_2_link" reason="Never" />
-    <disable_collisions link1="tool0" link2="wrist_3_link" reason="Adjacent" />
-    <disable_collisions link1="forearm_link" link2="upper_arm_link" reason="Adjacent" />
-    <disable_collisions link1="forearm_link" link2="wrist_1_link" reason="Adjacent" />
-    <disable_collisions link1="shoulder_link" link2="upper_arm_link" reason="Adjacent" />
-    <disable_collisions link1="wrist_1_link" link2="wrist_2_link" reason="Adjacent" />
-    <disable_collisions link1="wrist_1_link" link2="wrist_3_link" reason="Never" />
-    <disable_collisions link1="wrist_2_link" link2="wrist_3_link" reason="Adjacent" />
+    <disable_collisions link1="ur_base_link" link2="ur_base_link_inertia" reason="Adjacent" />
+    <disable_collisions link1="ur_base_link_inertia" link2="ur_shoulder_link" reason="Adjacent" />
+    <disable_collisions link1="ur_tool0" link2="ur_wrist_1_link" reason="Never" />
+    <disable_collisions link1="ur_tool0" link2="ur_wrist_2_link" reason="Never" />
+    <disable_collisions link1="ur_tool0" link2="ur_wrist_3_link" reason="Adjacent" />
+    <disable_collisions link1="ur_forearm_link" link2="ur_upper_arm_link" reason="Adjacent" />
+    <disable_collisions link1="ur_forearm_link" link2="ur_wrist_1_link" reason="Adjacent" />
+    <disable_collisions link1="ur_shoulder_link" link2="ur_upper_arm_link" reason="Adjacent" />
+    <disable_collisions link1="ur_wrist_1_link" link2="ur_wrist_2_link" reason="Adjacent" />
+    <disable_collisions link1="ur_wrist_1_link" link2="ur_wrist_3_link" reason="Never" />
+    <disable_collisions link1="ur_wrist_2_link" link2="ur_wrist_3_link" reason="Adjacent" />
   </xacro:macro>
 </robot>
